Commit message: add oakd cameara into sim robot

File: src/simulation/urdf/my_robot.urdf (robot description, URDF)
Before this commit: robot my_robot, 5 links, 4 joints
Links:
- added link oakd_link, mass 0.05; collision box size=0.02 0.09 0.02; visual box size=0.02 0.09 0.02
- added link oakd_rgb_camera_frame
- added link oakd_rgb_camera_optical_frame
Joints:
- added joint oakd_joint: type fixed, parent base_link, child oakd_link, origin xyz=0.30 0 0.05 rpy=0 0 0
- added joint oakd_rgb_camera_joint: type fixed, parent oakd_link, child oakd_rgb_camera_frame, origin xyz=0.01 0 0 rpy=0 0 0
- added joint oakd_rgb_camera_optical_joint: type fixed, parent oakd_rgb_camera_frame, child oakd_rgb_camera_optical_frame, origin xyz=0 0 0 rpy=-1.5707963 0 -1.5707963
